Commit message: Got visualization working

File: mote_control/description/ros2_control/mote.ros2_control.xacro (robot description, xacro)
@@ -1,5 +1,5 @@
 <?xml version="1.0"?>
 <robot xmlns:xacro="http://www.ros.org/wiki/xacro">
-  <xacro:macro name="mote_control" params="name prefix use_mock_hardware">
+  <xacro:macro name="mote_ros2_control" params="name prefix use_mock_hardware">
     <ros2_control name="${name}" type="system">
       <xacro:unless value="${use_mock_hardware}">

File: mote_control/description/urdf/mote.urdf.xacro (robot description, xacro)
@@ -1,14 +1,14 @@
 <?xml version="1.0"?>
 <!-- Basic differential drive mobile base -->
-<robot xmlns:xacro="http://www.ros.org/wiki/xacro" name="diffdrive_robot">
+<robot xmlns:xacro="http://www.ros.org/wiki/xacro" name="mote_robot">
   <xacro:arg name="prefix" default="" />
-  <xacro:arg name="use_mock_hardware" default="false" />
-  <xacro:include filename="$(find ros2_control_demo_description)/diffbot/urdf/diffbot_description.urdf.xacro" />
+  <xacro:arg name="use_mock_hardware" default="true" />
+  <xacro:include filename="$(find mote_description)/mote/urdf/mote.urdf.xacro" />
   <!-- Import Rviz colors -->
-  <!-- <xacro:include filename="$(find ros2_control_demo_description)/diffbot/urdf/diffbot.materials.xacro" /> -->
+  <xacro:include filename="$(find mote_description)/mote/urdf/mote.materials.xacro" />
   <!-- Import mote ros2_control description -->
-  <xacro:include filename="$(find mote_control)/ros2_control/diffbot.ros2_control.xacro" />
-  <xacro:diffbot prefix="$(arg prefix)" />
-  <xacro:diffbot_ros2_control
+  <xacro:include filename="$(find mote_control)/ros2_control/mote.ros2_control.xacro" />
+  <xacro:mote prefix="$(arg prefix)" />
+  <xacro:mote_ros2_control
     name="Mote" prefix="$(arg prefix)" use_mock_hardware="$(arg use_mock_hardware)"/>
 </robot>
